File: Link Robotics 5G.kicad_sch (KiCad schematic)
At the start: 119 parts, among them J1 T1, J10 Nano SIM, J11 T4, J2 T2, J3 T3, J4 T4, J5 T5, J6 T6, J7 1714936, J8 Conn_U.FL, J9 2199230-3, Q1 NTR4501, Q2 NTR4501, Q3 NTR4501, Q4 BSS138, Q5 BSS138, Q6 BSS138, Q7 BSS138, Q8 BSS138, Q9 BSS138, SW1 SW_DPDT_x2, SW2 SW_Push, U1 LF33_TO252, U2 SPX3819M5-L-3-3, U3 LM2678, U4 LD39015M18R, U5 ZED-F9P, U6 STM32F415RGTx, U7 PE1805C4A6, Y1 16MHZ

Commit message: Add files via upload
27.10.2022
Parts:
- removed Q2: NTR4501, Package_TO_SOT_SMD:SOT-23, symbol Transistor_FET:2N7002
- removed R10: 30K, symbol Device:R_Small
- added Q?: BSS138, Package_TO_SOT_SMD:SOT-23, symbol Transistor_FET:BSS138
Connections:
- net GND: now also Q?.2 (S)
- net Vsw_on/off: now also Q?.1 (G)
- net at R5.1, U2.3 (EN): now also Q?.3 (D)
Changed lines of the file:
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@@
   (junction (at 80.772 56.2356) (diameter 0) (color 0 0 0 0)
   )
-  (junction (at 88.773 101.8794) (diameter 0) (color 0 0 0 0)
-  )
   (junction (at 50.2666 94.2594) (diameter 0) (color 0 0 0 0)
   )
@@
   (junction (at 207.6704 163.957) (diameter 0) (color 0 0 0 0)
   )
-  (junction (at 88.773 112.0394) (diameter 0) (color 0 0 0 0)
-  )
   (junction (at 268.0208 39.2176) (diameter 0) (color 0 0 0 0)
   )
@@
     (stroke (width 0) (type default) (color 0 0 0 0))
   )
-  (wire (pts (xy 88.773 104.4194) (xy 88.773 101.8794))
-    (stroke (width 0) (type default) (color 0 0 0 0))
-  )
   (wire (pts (xy 372.0846 186.1058) (xy 369.9002 186.1058))
     (stroke (width 0) (type default) (color 0 0 0 0))
@@
     (stroke (width 0) (type default) (color 0 0 0 0))
   )
-  (wire (pts (xy 88.773 109.4994) (xy 88.773 112.0394))
-    (stroke (width 0) (type default) (color 0 0 0 0))
-  )
   (wire (pts (xy 48.5902 40.9956) (xy 48.5902 46.0756))
     (stroke (width 0) (type default) (color 0 0 0 0))
@@
     (stroke (width 0) (type default) (color 0 0 0 0))
   )
-  (wire (pts (xy 88.773 112.0394) (xy 68.453 112.0394))
-    (stroke (width 0) (type default) (color 0 0 0 0))
-  )
   (wire (pts (xy 95.4786 72.136) (xy 100.5586 72.136))
     (stroke (width 0) (type default) (color 0 0 0 0))
@@
     (stroke (width 0) (type default) (color 0 0 0 0))
   )
-  (wire (pts (xy 101.473 112.0394) (xy 88.773 112.0394))
+  (wire (pts (xy 68.453 112.0394) (xy 101.473 112.0394))
     (stroke (width 0) (type default) (color 0 0 0 0))
   )
@@
     (pin "1")
   )
-  (symbol (lib_id "Device:R_Small") (at 88.773 106.9594 180) (unit 1)
-    (in_bom yes) (on_board yes)
-    (property "Reference" "R10" (id 0) (at 89.9668 105.8418 0)
-      (effects (font (size 1.27 1.27)) (justify right))
-    )
-    (property "Value" "30K" (id 1) (at 89.9668 108.3818 0)
-      (effects (font (size 1.27 1.27)) (justify right))
-    )
-    (property "Footprint" "" (id 2) (at 88.773 106.9594 0)
-      (effects (font (size 1.27 1.27)) hide)
-    )
-    (property "Datasheet" "~" (id 3) (at 88.773 106.9594 0)
-      (effects (font (size 1.27 1.27)) hide)
-    )
-    (pin "1")
-    (pin "2")
-  )
   (symbol (lib_id "Device:R_Small") (at 354.3554 37.1094 0) (unit 1)
     (in_bom yes) (on_board yes)
@@
     (pin "1")
   )
-  (symbol (lib_id "Transistor_FET:2N7002") (at 57.0738 104.394 0) (mirror x) (unit 1)
-    (in_bom yes) (on_board yes)
-    (property "Reference" "Q2" (id 0) (at 60.1472 108.077 0)
-      (effects (font (size 1.27 1.27)) (justify left))
-    )
-    (property "Value" "NTR4501" (id 1) (at 51.0286 109.7788 0)
-      (effects (font (size 1.27 1.27)) (justify left))
-    )
-    (property "Footprint" "Package_TO_SOT_SMD:SOT-23" (id 2) (at 62.1538 102.489 0)
-      (effects (font (size 1.27 1.27) italic) (justify left) hide)
-    )
-    (property "Datasheet" "https://www.digikey.com/en/products/detail/onsemi/NTR4501NST1G/4848850" (id 3) (at 57.0738 104.394 0)
-      (effects (font (size 1.27 1.27)) (justify left) hide)
-    )
-    (pin "1")
-    (pin "2")
-    (pin "3")
-  )
   (symbol (lib_id "Device:C_Small") (at 176.8602 167.132 0) (unit 1)
     (in_bom yes) (on_board yes)
@@
     (pin "1")
   )
+  (symbol (lib_id "Transistor_FET:BSS138") (at 57.0738 104.394 0) (unit 1)
+    (in_bom yes) (on_board yes)
+    (property "Reference" "Q?" (id 0) (at 54.8386 102.3112 90))
+    (property "Value" "BSS138" (id 1) (at 63.2714 104.1908 90))
+    (property "Footprint" "Package_TO_SOT_SMD:SOT-23" (id 2) (at 62.1538 106.299 0)
+      (effects (font (size 1.27 1.27) italic) (justify left) hide)
+    )
+    (property "Datasheet" "https://ozdisan.com/power-semiconductors/mosfets/discrete-mosfets/BSS138-HT" (id 3) (at 57.0738 104.394 0)
+      (effects (font (size 1.27 1.27)) (justify left) hide)
+    )
+    (pin "1")
+    (pin "2")
+    (pin "3")
+  )
   (symbol (lib_id "Device:R_Small") (at 179.7304 246.2022 270) (unit 1)
     (in_bom yes) (on_board yes)
@@
       (reference "Q1") (unit 1) (value "NTR4501") (footprint "Package_TO_SOT_SMD:SOT-23")
     )
-    (path "/79a0cabe-aea3-4d04-a846-73da0b530c18"
-      (reference "Q2") (unit 1) (value "NTR4501") (footprint "Package_TO_SOT_SMD:SOT-23")
-    )
     (path "/429025d5-3235-4978-8071-a3b79cc29c40"
       (reference "Q3") (unit 1) (value "NTR4501") (footprint "Package_TO_SOT_SMD:SOT-23")
@@
       (reference "Q9") (unit 1) (value "BSS138") (footprint "Package_TO_SOT_SMD:SOT-23")
     )
+    (path "/ef9fe295-ec16-4167-b32f-cc8c38ba2b8c"
+      (reference "Q?") (unit 1) (value "BSS138") (footprint "Package_TO_SOT_SMD:SOT-23")
+    )
     (path "/af9a412e-ea77-4bf4-9513-5e9d44b4410f"
       (reference "R1") (unit 1) (value "10K") (footprint "")
@@
       (reference "R9") (unit 1) (value "50K") (footprint "")
     )
-    (path "/634a41cf-dde4-4dbd-9ee8-b4f0c28e2a32"
-      (reference "R10") (unit 1) (value "30K") (footprint "")
-    )
     (path "/5a6c73ff-ca49-4c73-9096-ccbff3b17bcb"
